Commit message: Finish hand model

File: teste_description/urdf/teste.urdf.xacro (robot description, xacro)
@@ -1,8 +1,9 @@
 <?xml version="1.0" ?>
 <robot name="elir_test" xmlns:xacro="http://www.ros.org/wiki/xacro">
+<xacro:property name="M_PI" value="3.141592" />
   <link name="base_link">
   </link>
-  <joint name="base_joint" type="fixed">
-    <origin xyz="0.0 0.0 0.025" rpy="0.0 0.0 0.0"/>
+  <joint name="world_base_joint" type="fixed">
+    <origin xyz="0.0 0.0 0.0" rpy="0.0 0.0 0.0"/>
     <parent link="base_link"/>
     <child link="zord_link0"/>
@@ -10,16 +11,104 @@
     <link name="zord_link0">
     <!-- This visual represents the base body-->
-    <visual name = 'base_body'>
+    <visual>
       <geometry>
         <cylinder length="0.05" radius="0.2"/>
       </geometry>
-      <material name="grey"/>
     </visual>
-    <collision name = 'base_body'>
+    <collision>
       <geometry>
-        <cylinder length="0.05" radius="0.2"/>
+        <cylinder length="0.02" radius="0.2"/>
       </geometry>
       <origin rpy="0 0 0" xyz="0.0 0.0 0"/>
     </collision>
     </link>
+    <joint name="joint_0" type="revolute">
+      <parent link="zord_link0"/>
+      <child link="zord_link1"/>
+      <origin rpy="0 0 0" xyz="0 0 0.025"/>
+      <limit effort="1000.0" lower="-3.14" upper="3.14" velocity="0.5"/>
+      <axis xyz="0 0 1"/>
+    </joint>
+    <link name="zord_link1">
+      <!-- This visual represents the base body-->
+    <visual>
+      <geometry>
+        <cylinder length="0.3" radius="0.01"/>
+      </geometry>
+      <origin rpy="0 0 0" xyz="0.0 0.0 0.15"/>
+    </visual>
+    <collision>
+      <geometry>
+        <cylinder length="0.2" radius="0.01"/>
+      </geometry>
+      <origin rpy="0 0 0" xyz="0.0 0.0 0.1"/>
+    </collision>
+    </link>
+    <joint name="joint_1" type="revolute">
+      <parent link="zord_link1"/>
+      <child link="zord_link2"/>
+      <origin rpy="0 0 0" xyz="0 0 0.3"/>
+      <limit effort="1000.0" lower="-3.14" upper="3.14" velocity="0.5"/>
+      <axis xyz="0 1 0"/>
+    </joint>
+    <link name="zord_link2">
+      <!-- This visual represents the base body-->
+    <visual>
+      <geometry>
+        <cylinder length="0.3" radius="0.01"/>
+      </geometry>
+      <origin rpy="0 0 0" xyz="0.0 0.0 0.15"/>
+    </visual>
+    <collision>
+      <geometry>
+        <cylinder length="0.2" radius="0.01"/>
+      </geometry>
+      <origin rpy="0 0 0" xyz="0.0 0.0 0.1"/>
+    </collision>
+    </link>
+    <joint name="joint_2" type="revolute">
+      <parent link="zord_link2"/>
+      <child link="zord_link3"/>
+      <origin rpy="0 0 0" xyz="0 0 0.3"/>
+      <limit effort="1000.0" lower="-3.14" upper="3.14" velocity="0.5"/>
+      <axis xyz="0 1 0"/>
+    </joint>
+    <link name="zord_link3">
+      <!-- This visual represents the base body-->
+    <visual>
+      <geometry>
+        <cylinder length="0.3" radius="0.01"/>
+      </geometry>
+      <origin rpy="0 0 0" xyz="0.0 0.0 0.15"/>
+    </visual>
+    <collision>
+      <geometry>
+        <cylinder length="0.2" radius="0.01"/>
+      </geometry>
+      <origin rpy="0 0 0" xyz="0.0 0.0 0.1"/>
+    </collision>
+    </link>
+    <joint name="joint_hqne" type="revolute">
+      <parent link="zord_link3"/>
+      <child link="zord_hand"/>
+      <origin rpy="0 0 0" xyz="0.015 0 ${0.3}"/>
+      <limit effort="1000.0" lower="-3.14" upper="3.14" velocity="0.5"/>
+      <axis xyz="1 0 0"/>
+    </joint>
+    <link name="zord_hand">
+    <visual>
+      <geometry>
+        <mesh filename="package://teste_description/meshes/Hand_Victory.stl" scale="0.002 0.002 0.002"/>
+      </geometry>
+      <material name="grey"/>
+      <origin rpy="0 0 0" xyz="0.0 0.0 ${0.06+0.043}"/>
+    </visual>
+    <!-- this collision is for the front f1 claw unit -->
+    <collision>
+      <geometry>
+        <mesh filename="package://teste_description/meshes/Hand_Victory.stl" scale="0.002 0.002 0.002" />
+      </geometry>
+      <origin rpy="0 0 0" xyz="0.0 0.0 ${0.06+0.043}"/>
+    </collision>
+  </link>
 </robot>
