Commit message: firsts tests with move it

File: victory_description/urdf/victory.urdf.xacro (robot description, xacro)
@@ -2,4 +2,13 @@
 <robot name="elir_test" xmlns:xacro="http://www.ros.org/wiki/xacro">
 <xacro:property name="M_PI" value="3.141592" />
+  <material name="purple">
+    <color rgba="${153/255} ${90/255} ${255/255} 1.0"/>
+  </material>
+  <material name="blue">
+    <color rgba="${90/255} ${129/255} ${255/255} 1.0"/>
+  </material>
+  <material name="light_blue">
+    <color rgba="${90/255} ${255/255} ${217/255} 1.0"/>
+  </material>
   <link name="base_link">
   </link>
@@ -7,7 +16,7 @@
     <origin xyz="0.0 0.0 0.0" rpy="0.0 0.0 0.0"/>
     <parent link="base_link"/>
-    <child link="zord_link0"/>
+    <child link="victory_link0"/>
   </joint>
-    <link name="zord_link0">
+    <link name="victory_link0">
     <!-- This visual represents the base body-->
     <visual>
@@ -15,4 +24,5 @@
         <cylinder length="0.05" radius="0.2"/>
       </geometry>
+      <material name="purple"/>
     </visual>
     <collision>
@@ -24,11 +34,11 @@
     </link>
     <joint name="joint_0" type="revolute">
-      <parent link="zord_link0"/>
-      <child link="zord_link1"/>
+      <parent link="victory_link0"/>
+      <child link="victory_link1"/>
       <origin rpy="0 0 0" xyz="0 0 0.025"/>
       <limit effort="1000.0" lower="-3.14" upper="3.14" velocity="0.5"/>
       <axis xyz="0 0 1"/>
     </joint>
-    <link name="zord_link1">
+    <link name="victory_link1">
       <!-- This visual represents the base body-->
     <visual>
@@ -37,4 +47,5 @@
       </geometry>
       <origin rpy="0 0 0" xyz="0.0 0.0 0.15"/>
+      <material name="blue"/>
     </visual>
     <collision>
@@ -46,11 +57,11 @@
     </link>
     <joint name="joint_1" type="revolute">
-      <parent link="zord_link1"/>
-      <child link="zord_link2"/>
+      <parent link="victory_link1"/>
+      <child link="victory_link2"/>
       <origin rpy="0 0 0" xyz="0 0 0.3"/>
       <limit effort="1000.0" lower="-3.14" upper="3.14" velocity="0.5"/>
       <axis xyz="0 1 0"/>
     </joint>
-    <link name="zord_link2">
+    <link name="victory_link2">
       <!-- This visual represents the base body-->
     <visual>
@@ -59,4 +70,5 @@
       </geometry>
       <origin rpy="0 0 0" xyz="0.0 0.0 0.15"/>
+      <material name="blue"/>
     </visual>
     <collision>
@@ -68,11 +80,11 @@
     </link>
     <joint name="joint_2" type="revolute">
-      <parent link="zord_link2"/>
-      <child link="zord_link3"/>
+      <parent link="victory_link2"/>
+      <child link="victory_link3"/>
       <origin rpy="0 0 0" xyz="0 0 0.3"/>
       <limit effort="1000.0" lower="-3.14" upper="3.14" velocity="0.5"/>
       <axis xyz="0 1 0"/>
     </joint>
-    <link name="zord_link3">
+    <link name="victory_link3">
       <!-- This visual represents the base body-->
     <visual>
@@ -81,4 +93,5 @@
       </geometry>
       <origin rpy="0 0 0" xyz="0.0 0.0 0.15"/>
+      <material name="blue"/>
     </visual>
     <collision>
@@ -89,23 +102,30 @@
     </collision>
     </link>
-    <joint name="joint_hqne" type="revolute">
-      <parent link="zord_link3"/>
-      <child link="zord_hand"/>
-      <origin rpy="0 0 0" xyz="0.015 0 ${0.3}"/>
-      <limit effort="1000.0" lower="-3.14" upper="3.14" velocity="0.5"/>
+    <joint name="joint_ref" type="fixed">
+      <parent link="victory_link3"/>
+      <child link="victory_ref"/>
+      <origin rpy="0 0 0" xyz="0 0 ${0.3}"/>
+      <axis xyz="0 0 0"/>
+    </joint>
+    <link name="victory_ref"/>
+    <joint name="joint_hand" type="revolute">
+      <parent link="victory_ref"/>
+      <child link="victory_hand"/>
+      <origin rpy="0 0 0" xyz="0.0 0.0 0.0"/>
+      <limit effort="1000.0" lower="${-M_PI/2}" upper="${M_PI/2}" velocity="0.5"/>
       <axis xyz="1 0 0"/>
     </joint>
-    <link name="zord_hand">
+    <link name="victory_hand">
     <visual>
       <geometry>
-        <mesh filename="package://teste_description/meshes/Hand_Victory.stl" scale="0.002 0.002 0.002"/>
+        <mesh filename="package://victory_description/meshes/Hand_Victory.stl" scale="0.002 0.002 0.002"/>
       </geometry>
-      <material name="grey"/>
-      <origin rpy="0 0 0" xyz="0.0 0.0 ${0.06+0.043}"/>
+      <material name="light_blue"/>
+      <origin rpy="0 0 0" xyz="0.015 0.0 ${0.06+0.043}"/>
     </visual>
     <!-- this collision is for the front f1 claw unit -->
     <collision>
       <geometry>
-        <mesh filename="package://teste_description/meshes/Hand_Victory.stl" scale="0.002 0.002 0.002" />
+        <mesh filename="package://victory_description/meshes/Hand_Victory.stl" scale="0.002 0.002 0.002" />
       </geometry>
       <origin rpy="0 0 0" xyz="0.0 0.0 ${0.06+0.043}"/>

Commit message: remove base_link

File: victory_description/urdf/victory.urdf.xacro (robot description, xacro)
@@ -11,5 +11,5 @@
     <color rgba="${90/255} ${255/255} ${217/255} 1.0"/>
   </material>
-  <link name="base_link">
+  <!-- <link name="base_link">
   </link>
   <joint name="world_base_joint" type="fixed">
@@ -17,5 +17,5 @@
     <parent link="base_link"/>
     <child link="victory_link0"/>
-  </joint>
+  </joint> -->
     <link name="victory_link0">
     <!-- This visual represents the base body-->
@@ -109,9 +109,8 @@
     </joint>
     <link name="victory_ref"/>
-    <joint name="joint_hand" type="revolute">
+    <joint name="joint_hand" type="fixed">
       <parent link="victory_ref"/>
       <child link="victory_hand"/>
       <origin rpy="0 0 0" xyz="0.0 0.0 0.0"/>
-      <limit effort="1000.0" lower="${-M_PI/2}" upper="${M_PI/2}" velocity="0.5"/>
       <axis xyz="1 0 0"/>
     </joint>
